File: hardware/zxuno.brd (EAGLE design)
At the start: 86 x 56 mm, 103 parts, among them T1 BC846, U1 6SLX9TQG144, U2 FLASH-SPI-25XXSMD1, U4 AD724, U5 50MHz, U6 3.3V, U7 1.2V, Y1 3.58M, Y2 4.43M

Commit message: Últimos cambios, probablemente sea v4.2 definitiva
Parts:
- renumbered JP1 to JTAG, JP2 to KEYB
Connections:
- net CLKPS2: no longer KEYB.1
- net DATAPS2: no longer KEYB.2
- net PS2_CLK: now also KEYB.2
- net PS2_DATA: now also KEYB.1
Routing:
- net DATAPS2: track 17.8 -> 6.99 mm
- net PS2_DATA: track 29.6 -> 37.8 mm
- net CLKPS2: track 9.29 -> 4.42 mm
- net PS2_CLK: track 27.4 -> 31.1 mm
- net N$15: track 27.2 -> 29.6 mm
Other:
- board text added: "v4.2"
- board text removed: "J16"
- board text removed: "JTAG"
- board text removed: "v4.1"
Changed lines of the file:
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@@
 <text x="0.76195" y="53.530421875" size="1.016" layer="25" font="vector" ratio="15">1</text>
 <text x="0.78310625" y="48.386946875" size="1.016" layer="25" font="vector" ratio="15">1</text>
-<text x="24.3331875" y="35.151484375" size="1.016" layer="21" font="vector" ratio="15">v4.1</text>
+<text x="24.3331875" y="35.151484375" size="1.016" layer="21" font="vector" ratio="15">v4.2</text>
 <text x="1.447325" y="42.234396875" size="1.016" layer="21" font="vector" ratio="15">(C)2015 ZX-Uno Team
 http://www.zxuno.com</text>
@@
 <rectangle x1="19.124090625" y1="39.578759375" x2="22.319409375" y2="39.599840625" layer="21"/>
 <text x="46.0375" y="26.7096875" size="1" layer="26" font="vector" ratio="15" rot="MR270">1</text>
-<text x="64.373125" y="18.3753125" size="1" layer="26" font="vector" ratio="15" rot="MR0">1</text>
+<text x="70.4903125" y="18.9221875" size="1" layer="26" font="vector" ratio="15" rot="MR0">1</text>
 <text x="24.765" y="5.953125" size="1" layer="25" font="vector" ratio="15">1</text>
 <text x="39.0525" y="0.9525" size="1" layer="26" font="vector" ratio="15" rot="MR0">1</text>
@@
 <text x="31.323078125" y="51.017271875" size="1.016" layer="125" font="vector" ratio="15">J11</text>
 <text x="32.52904375" y="48.39294375" size="1.016" layer="125" font="vector" ratio="15">J12</text>
-<text x="65.88125" y="18.176875" size="1.016" layer="125" font="vector" ratio="15" rot="R270">J16</text>
 <text x="73.57231875" y="17.811725" size="1.016" layer="125" font="vector" ratio="15">JOY</text>
-<text x="58.09249375" y="16.2298375" size="1.016" layer="125" font="vector" ratio="15">JTAG</text>
 <text x="3.0916625" y="27.65549375" size="1.016" layer="125" font="vector" ratio="15">L1</text>
 <text x="21.55825" y="30.8014625" size="1.016" layer="125" font="vector" ratio="15" rot="R90">L2</text>
@@
 <attribute name="NAME" x="40.86671875" y="45.7596875" size="1.016" layer="25" font="vector" ratio="15" rot="R180"/>
 </element>
-<element name="JP1" library="pinhead" package="1X06" value="" x="61.921875" y="18.734375" rot="R180"/>
-<element name="JP2" library="pinhead" package="1X03" value="" x="68.265625" y="16.1953125" rot="R180"/>
+<element name="JTAG" library="pinhead" package="1X06" value="" x="61.921875" y="18.734375" smashed="yes" rot="R180">
+<attribute name="NAME" x="61.4383875" y="17.3352625" size="1.016" layer="125" font="vector" ratio="15" rot="R180"/>
+<attribute name="VALUE" x="69.541875" y="21.909375" size="1.27" layer="27" rot="R180"/>
+</element>
+<element name="KEYB" library="pinhead" package="1X03" value="" x="68.265625" y="16.1953125" smashed="yes" rot="R180">
+<attribute name="NAME" x="72.6987" y="18.5462" size="1.016" layer="125" font="vector" ratio="15" rot="R180"/>
+<attribute name="VALUE" x="72.075625" y="19.3703125" size="1.27" layer="27" rot="R180"/>
+</element>
 </elements>
 <signals>
@@
 <wire x1="53.75671875" y1="35.06390625" x2="52.85859375" y2="35.06390625" width="0.1778" layer="1"/>
 <wire x1="52.85859375" y1="35.06390625" x2="52.85125" y2="35.07125" width="0.1778" layer="1"/>
-<contactref element="JP1" pad="2"/>
+<contactref element="JTAG" pad="2"/>
 </signal>
 <signal name="XD0">
@@
 <wire x1="41.91" y1="4.355625" x2="43.581" y2="2.684625" width="0.2032" layer="1"/>
 <wire x1="43.581" y1="2.04375" x2="43.581" y2="2.684625" width="0.2032" layer="1"/>
-<contactref element="JP1" pad="1"/>
+<contactref element="JTAG" pad="1"/>
 <wire x1="68.271875" y1="18.734375" x2="68.271875" y2="21.028125" width="0.3048" layer="16"/>
 <wire x1="68.271875" y1="21.028125" x2="66.46625" y2="22.83375" width="0.3048" layer="16"/>
@@
 <wire x1="68.42125" y1="9.36625" x2="68.42125" y2="10.63625" width="0.1778" layer="1"/>
 <wire x1="68.42125" y1="10.63625" x2="63.8175" y2="15.24" width="0.1778" layer="1"/>
+<contactref element="KEYB" pad="1"/>
+<wire x1="70.805625" y1="16.1953125" x2="70.805625" y2="16.180625" width="0.1778" layer="1"/>
+<wire x1="70.805625" y1="16.180625" x2="70.34375" y2="15.71875" width="0.1778" layer="1"/>
+<wire x1="70.34375" y1="15.71875" x2="70.34375" y2="9.54" width="0.1778" layer="1"/>
+<wire x1="70.34375" y1="9.54" x2="69.37625" y2="8.5725" width="0.1778" layer="1"/>
 </signal>
 <signal name="PS2_CLK">
@@
 <wire x1="46.00125" y1="18.2925" x2="48.73625" y2="15.5575" width="0.1778" layer="1"/>
 <wire x1="69.37625" y1="10.795" x2="68.8975" y2="10.795" width="0.1778" layer="1"/>
-<wire x1="68.8975" y1="10.795" x2="64.135" y2="15.5575" width="0.1778" layer="1"/>
+<contactref element="KEYB" pad="2"/>
+<wire x1="64.135" y1="15.5575" x2="64.135" y2="15.5525" width="0.1778" layer="1"/>
+<wire x1="64.135" y1="15.5525" x2="65.171875" y2="14.515625" width="0.1778" layer="1"/>
+<wire x1="68.265625" y1="16.1953125" x2="68.265625" y2="14.515625" width="0.1778" layer="1"/>
+<wire x1="68.265625" y1="14.515625" x2="68.265625" y2="11.905625" width="0.1778" layer="1"/>
+<wire x1="68.265625" y1="11.905625" x2="69.37625" y2="10.795" width="0.1778" layer="1"/>
+<wire x1="65.171875" y1="14.515625" x2="68.265625" y2="14.515625" width="0.1778" layer="1"/>
 </signal>
 <signal name="EAR">
@@
 <contactref element="U1" pad="P109"/>
 <wire x1="52.85125" y1="21.57125" x2="60.355" y2="21.57125" width="0.1778" layer="1"/>
-<contactref element="JP1" pad="3"/>
+<contactref element="JTAG" pad="3"/>
 <wire x1="60.355" y1="21.57125" x2="63.191875" y2="18.734375" width="0.1778" layer="1"/>
 </signal>
@@
 <wire x1="49.50125" y1="18.285" x2="50.32375" y2="17.4625" width="0.1778" layer="1"/>
 <wire x1="50.32375" y1="17.4625" x2="59.38" y2="17.4625" width="0.1778" layer="1"/>
-<contactref element="JP1" pad="4"/>
+<contactref element="JTAG" pad="4"/>
 <wire x1="59.38" y1="17.4625" x2="60.651875" y2="18.734375" width="0.1778" layer="1"/>
 </signal>
@@
 <wire x1="52.85125" y1="22.07125" x2="51.519375" y2="22.07125" width="0.1778" layer="1"/>
 <wire x1="51.519375" y1="22.07125" x2="51.1571875" y2="21.7090625" width="0.1778" layer="1"/>
-<contactref element="JP1" pad="5"/>
+<contactref element="JTAG" pad="5"/>
 <wire x1="51.1571875" y1="21.7090625" x2="51.1571875" y2="20.7490625" width="0.1778" layer="1"/>
 <wire x1="51.1571875" y1="20.7490625" x2="51.9296875" y2="20.0078125" width="0.1778" layer="1"/>
@@
 <wire x1="39.3620625" y1="43.6959375" x2="33.147" y2="49.911" width="0.3048" layer="16"/>
 <contactref element="R5" pad="1"/>
-<contactref element="JP2" pad="3"/>
+<contactref element="KEYB" pad="3"/>
 <wire x1="65.725625" y1="16.1953125" x2="65.725625" y2="16.1728125" width="0.3048" layer="16"/>
 <wire x1="65.725625" y1="16.1728125" x2="67.015625" y2="14.8828125" width="0.3048" layer="16"/>
 <wire x1="67.015625" y1="14.8828125" x2="68.9816375" y2="14.8828125" width="0.3048" layer="16"/>
 <wire x1="68.9816375" y1="14.8828125" x2="77.05725" y2="6.8072" width="0.3048" layer="16"/>
-<wire x1="71.755" y1="13.0175" x2="71.27625" y2="13.0175" width="0" layer="19" extent="1-1"/>
+<wire x1="71.755" y1="13.0175" x2="71.27625" y2="13.0175" width="0.3048" layer="1"/>
 </signal>
 <signal name="N$14">
@@
 <wire x1="50.00125" y1="19.22125" x2="50.00125" y2="18.26125" width="0.1778" layer="1"/>
 <wire x1="50.00125" y1="18.26125" x2="50.4825" y2="17.78" width="0.1778" layer="1"/>
-<contactref element="JP1" pad="6"/>
+<contactref element="JTAG" pad="6"/>
 <wire x1="50.4825" y1="17.78" x2="54.6175" y2="17.78" width="0.1778" layer="1"/>
 <wire x1="54.6175" y1="17.78" x2="55.571875" y2="18.734375" width="0.1778" layer="1"/>
@@
 <wire x1="78.0615625" y1="33.2275" x2="79.6484375" y2="31.640625" width="0.1778" layer="1"/>
 <wire x1="79.6484375" y1="31.640625" x2="79.6484375" y2="20.7890625" width="0.1778" layer="1"/>
-<wire x1="79.6484375" y1="20.7890625" x2="74.7734375" y2="15.9140625" width="0.1778" layer="1"/>
-<wire x1="74.7734375" y1="15.9140625" x2="73.9296875" y2="15.9140625" width="0.1778" layer="1"/>
-<wire x1="73.9296875" y1="15.9140625" x2="72.2578125" y2="14.2421875" width="0.1778" layer="1"/>
-<wire x1="72.2578125" y1="14.2421875" x2="70.046875" y2="14.2421875" width="0.1778" layer="1"/>
-<wire x1="70.046875" y1="14.2421875" x2="69.4140625" y2="13.609375" width="0.1778" layer="1"/>
 <wire x1="69.4140625" y1="13.609375" x2="69.4140625" y2="13.0553125" width="0.1778" layer="1"/>
 <wire x1="69.4140625" y1="13.0553125" x2="69.37625" y2="13.0175" width="0.1778" layer="1"/>
+<wire x1="79.6484375" y1="20.7890625" x2="76.3203125" y2="17.4609375" width="0.1778" layer="1"/>
+<wire x1="76.3203125" y1="17.4609375" x2="70.203125" y2="17.4609375" width="0.1778" layer="1"/>
+<wire x1="70.203125" y1="17.4609375" x2="69.5" y2="16.7578125" width="0.1778" layer="1"/>
+<wire x1="69.5" y1="16.7578125" x2="69.5" y2="13.14125" width="0.1778" layer="1"/>
+<wire x1="69.5" y1="13.14125" x2="69.37625" y2="13.0175" width="0.1778" layer="1"/>
 </signal>
 <signal name="DATAPS2">
@@
 <wire x1="74.70875" y1="11.495" x2="76.8614" y2="11.495" width="0.3048" layer="1"/>
 <wire x1="76.8614" y1="11.495" x2="77.05725" y2="11.4554" width="0.3048" layer="1"/>
-<contactref element="JP2" pad="2"/>
-<wire x1="68.265625" y1="16.1953125" x2="69.0078125" y2="16.1953125" width="0.3048" layer="16"/>
-<wire x1="69.0078125" y1="16.1953125" x2="73.75" y2="11.484375" width="0.3048" layer="16"/>
-<wire x1="73.75" y1="11.484375" x2="77.059525" y2="11.484375" width="0.3048" layer="16"/>
-<wire x1="77.059525" y1="11.484375" x2="77.05725" y2="11.4554" width="0.3048" layer="16"/>
 </signal>
 <signal name="CLKPS2">
@@
 <wire x1="71.27625" y1="10.795" x2="71.85025" y2="10.795" width="0.3048" layer="1"/>
 <wire x1="71.85025" y1="10.795" x2="74.56805" y2="13.5128" width="0.3048" layer="1"/>
-<contactref element="JP2" pad="1"/>
-<wire x1="70.805625" y1="16.1953125" x2="71.8855375" y2="16.1953125" width="0.3048" layer="16"/>
-<wire x1="71.8855375" y1="16.1953125" x2="74.56805" y2="13.5128" width="0.3048" layer="16"/>
 </signal>
 </signals>

Commit message: Cambios sugeridos por McLeod
Connections:
- net CLKPS2: now also KEYB.1
- net DATAPS2: now also KEYB.2
- net PS2_CLK: no longer KEYB.2
- net PS2_DATA: no longer KEYB.1
Routing:
- net DATAPS2: track 6.99 -> 17.7 mm
- net PS2_DATA: track 37.8 -> 29.6 mm
- net CLKPS2: track 4.42 -> 9.29 mm
- net PS2_CLK: track 31.1 -> 27.9 mm
- net N$15: track 29.6 -> 27.4 mm
Changed lines of the file:
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@@
 <wire x1="68.42125" y1="9.36625" x2="68.42125" y2="10.63625" width="0.1778" layer="1"/>
 <wire x1="68.42125" y1="10.63625" x2="63.8175" y2="15.24" width="0.1778" layer="1"/>
-<contactref element="KEYB" pad="1"/>
-<wire x1="70.805625" y1="16.1953125" x2="70.805625" y2="16.180625" width="0.1778" layer="1"/>
-<wire x1="70.805625" y1="16.180625" x2="70.34375" y2="15.71875" width="0.1778" layer="1"/>
-<wire x1="70.34375" y1="15.71875" x2="70.34375" y2="9.54" width="0.1778" layer="1"/>
-<wire x1="70.34375" y1="9.54" x2="69.37625" y2="8.5725" width="0.1778" layer="1"/>
 </signal>
 <signal name="PS2_CLK">
@@
 <wire x1="46.00125" y1="18.2925" x2="48.73625" y2="15.5575" width="0.1778" layer="1"/>
 <wire x1="69.37625" y1="10.795" x2="68.8975" y2="10.795" width="0.1778" layer="1"/>
-<contactref element="KEYB" pad="2"/>
 <wire x1="64.135" y1="15.5575" x2="64.135" y2="15.5525" width="0.1778" layer="1"/>
-<wire x1="64.135" y1="15.5525" x2="65.171875" y2="14.515625" width="0.1778" layer="1"/>
-<wire x1="68.265625" y1="16.1953125" x2="68.265625" y2="14.515625" width="0.1778" layer="1"/>
-<wire x1="68.265625" y1="14.515625" x2="68.265625" y2="11.905625" width="0.1778" layer="1"/>
-<wire x1="68.265625" y1="11.905625" x2="69.37625" y2="10.795" width="0.1778" layer="1"/>
-<wire x1="65.171875" y1="14.515625" x2="68.265625" y2="14.515625" width="0.1778" layer="1"/>
+<wire x1="64.135" y1="15.5525" x2="64.8515625" y2="14.8359375" width="0.1778" layer="1"/>
+<wire x1="64.8515625" y1="14.8359375" x2="65.171875" y2="14.515625" width="0.1778" layer="1"/>
+<wire x1="69.37625" y1="10.795" x2="68.8925" y2="10.795" width="0.1778" layer="1"/>
+<wire x1="68.8925" y1="10.795" x2="65.171875" y2="14.515625" width="0.1778" layer="1"/>
 </signal>
 <signal name="EAR">
@@
 <contactref element="R5" pad="1"/>
 <contactref element="KEYB" pad="3"/>
-<wire x1="65.725625" y1="16.1953125" x2="65.725625" y2="16.1728125" width="0.3048" layer="16"/>
-<wire x1="65.725625" y1="16.1728125" x2="67.015625" y2="14.8828125" width="0.3048" layer="16"/>
-<wire x1="67.015625" y1="14.8828125" x2="68.9816375" y2="14.8828125" width="0.3048" layer="16"/>
-<wire x1="68.9816375" y1="14.8828125" x2="77.05725" y2="6.8072" width="0.3048" layer="16"/>
 <wire x1="71.755" y1="13.0175" x2="71.27625" y2="13.0175" width="0.3048" layer="1"/>
+<wire x1="77.05725" y1="6.8072" x2="76.5443625" y2="6.8072" width="0.3048" layer="16"/>
+<wire x1="76.5443625" y1="6.8072" x2="73.7109375" y2="9.640625" width="0.3048" layer="16"/>
+<wire x1="73.7109375" y1="9.640625" x2="72.2803125" y2="9.640625" width="0.3048" layer="16"/>
+<wire x1="72.2803125" y1="9.640625" x2="65.725625" y2="16.1953125" width="0.3048" layer="16"/>
 </signal>
 <signal name="N$14">
@@
 <wire x1="69.4140625" y1="13.0553125" x2="69.37625" y2="13.0175" width="0.1778" layer="1"/>
 <wire x1="79.6484375" y1="20.7890625" x2="76.3203125" y2="17.4609375" width="0.1778" layer="1"/>
-<wire x1="76.3203125" y1="17.4609375" x2="70.203125" y2="17.4609375" width="0.1778" layer="1"/>
-<wire x1="70.203125" y1="17.4609375" x2="69.5" y2="16.7578125" width="0.1778" layer="1"/>
-<wire x1="69.5" y1="16.7578125" x2="69.5" y2="13.14125" width="0.1778" layer="1"/>
 <wire x1="69.5" y1="13.14125" x2="69.37625" y2="13.0175" width="0.1778" layer="1"/>
+<wire x1="76.3203125" y1="17.4609375" x2="74.7109375" y2="17.4609375" width="0.1778" layer="1"/>
+<wire x1="74.7109375" y1="17.4609375" x2="71.921875" y2="14.671875" width="0.1778" layer="1"/>
+<wire x1="71.921875" y1="14.671875" x2="70.4765625" y2="14.671875" width="0.1778" layer="1"/>
+<wire x1="70.4765625" y1="14.671875" x2="69.4140625" y2="13.609375" width="0.1778" layer="1"/>
 </signal>
 <signal name="DATAPS2">
@@
 <wire x1="74.70875" y1="11.495" x2="76.8614" y2="11.495" width="0.3048" layer="1"/>
 <wire x1="76.8614" y1="11.495" x2="77.05725" y2="11.4554" width="0.3048" layer="1"/>
+<contactref element="KEYB" pad="2"/>
+<wire x1="77.05725" y1="11.4554" x2="73.0055375" y2="11.4554" width="0.3048" layer="16"/>
+<wire x1="73.0055375" y1="11.4554" x2="68.265625" y2="16.1953125" width="0.3048" layer="16"/>
 </signal>
 <signal name="CLKPS2">
@@
 <wire x1="71.27625" y1="10.795" x2="71.85025" y2="10.795" width="0.3048" layer="1"/>
 <wire x1="71.85025" y1="10.795" x2="74.56805" y2="13.5128" width="0.3048" layer="1"/>
+<contactref element="KEYB" pad="1"/>
+<wire x1="74.56805" y1="13.5128" x2="73.4881375" y2="13.5128" width="0.3048" layer="16"/>
+<wire x1="73.4881375" y1="13.5128" x2="70.805625" y2="16.1953125" width="0.3048" layer="16"/>
 </signal>
 </signals>
