File: hardware/usb_blaster.sch (EAGLE design)
At the start: 19 parts, among them IC2 PIC18F14K50SO, X1 53047-06

Commit message: Actualizo USB Blaster
Parts:
- removed C1: 0.1u, rcl:C-USC0603K
- removed JP2: (no value), pinhead:PINHD-2X3
- added JP3: (no value), pinhead:PINHD-1X1
- JP1: device pinhead:PINHD-1X5 -> pinhead:PINHD-2X4
Connections:
- new net N$5: JP1.5, JP1.7
- net GND: no longer C1.2, JP2.3
- net N$3: now also JP1.6, JP1.8; no longer JP2.5, JP2.6
- net PGC: no longer JP2.1
- net PGD: no longer JP2.2
- net VCC: no longer C1.1, JP2.4
- net VPP: now also JP3.1; no longer JP1.5
Changed lines of the file:
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@@
 <part name="P+2" library="supply1" deviceset="VCC" device=""/>
 <part name="GND9" library="supply1" deviceset="GND" device=""/>
-<part name="C1" library="rcl" deviceset="C-US" device="C0603K" value="0.1u"/>
 <part name="C2" library="SparkFun" deviceset="CAP" device="0805" value="4.7u"/>
 <part name="C5" library="rcl" deviceset="C-US" device="C0603K" value="0.33u"/>
@@
 <part name="R11" library="SparkFun" deviceset="RESISTOR" device="0805-RES" value="100R"/>
 <part name="R9" library="SparkFun" deviceset="RESISTOR" device="0805-RES" value="100R"/>
-<part name="JP1" library="pinhead" deviceset="PINHD-1X5" device=""/>
-<part name="JP2" library="pinhead" deviceset="PINHD-2X3" device=""/>
 <part name="X1" library="con-molex" deviceset="53?-06" device="047"/>
+<part name="JP3" library="pinhead" deviceset="PINHD-1X1" device=""/>
+<part name="JP1" library="pinhead" deviceset="PINHD-2X4" device=""/>
 </parts>
 <sheets>
@@
 <instance part="P+2" gate="VCC" x="53.34" y="104.14"/>
 <instance part="GND9" gate="1" x="53.34" y="91.44"/>
-<instance part="C1" gate="G$1" x="60.96" y="99.06"/>
 <instance part="C2" gate="G$1" x="68.58" y="96.52"/>
 <instance part="C5" gate="G$1" x="139.7" y="66.04"/>
@@
 <instance part="R11" gate="G$1" x="114.3" y="53.34"/>
 <instance part="R9" gate="G$1" x="109.22" y="38.1"/>
-<instance part="JP1" gate="A" x="114.3" y="96.52"/>
-<instance part="JP2" gate="A" x="170.18" y="71.12" rot="R90"/>
 <instance part="X1" gate="-6" x="134.62" y="101.6"/>
 <instance part="X1" gate="-5" x="134.62" y="99.06"/>
@@
 <instance part="X1" gate="-2" x="134.62" y="91.44"/>
 <instance part="X1" gate="-1" x="134.62" y="88.9"/>
+<instance part="JP3" gate="G$1" x="114.3" y="91.44"/>
+<instance part="JP1" gate="A" x="172.72" y="71.12" rot="R90"/>
 </instances>
 <busses>
@@
 </segment>
 <segment>
-<wire x1="53.34" y1="93.98" x2="60.96" y2="93.98" width="0.1524" layer="91"/>
-<wire x1="68.58" y1="93.98" x2="60.96" y2="93.98" width="0.1524" layer="91"/>
-<junction x="60.96" y="93.98"/>
+<wire x1="68.58" y1="93.98" x2="53.34" y2="93.98" width="0.1524" layer="91"/>
 <pinref part="GND9" gate="1" pin="GND"/>
-<pinref part="C1" gate="G$1" pin="2"/>
 <pinref part="C2" gate="G$1" pin="2"/>
-</segment>
-<segment>
-<wire x1="104.14" y1="96.52" x2="111.76" y2="96.52" width="0.1524" layer="91"/>
-<label x="101.6" y="96.52" size="1.27" layer="95"/>
-<pinref part="JP1" gate="A" pin="3"/>
 </segment>
 <segment>
@@
 <wire x1="170.18" y1="68.58" x2="170.18" y2="60.96" width="0.1524" layer="91"/>
 <label x="170.18" y="58.42" size="1.778" layer="95"/>
-<pinref part="JP2" gate="A" pin="3"/>
+<pinref part="JP1" gate="A" pin="3"/>
 </segment>
 </net>
@@
 </segment>
 <segment>
-<wire x1="68.58" y1="101.6" x2="60.96" y2="101.6" width="0.1524" layer="91"/>
-<wire x1="60.96" y1="101.6" x2="53.34" y2="101.6" width="0.1524" layer="91"/>
-<junction x="60.96" y="101.6"/>
+<wire x1="68.58" y1="101.6" x2="53.34" y2="101.6" width="0.1524" layer="91"/>
 <pinref part="C2" gate="G$1" pin="1"/>
-<pinref part="C1" gate="G$1" pin="1"/>
 <pinref part="P+2" gate="VCC" pin="VCC"/>
-</segment>
-<segment>
-<wire x1="104.14" y1="93.98" x2="111.76" y2="93.98" width="0.1524" layer="91"/>
-<label x="101.6" y="93.98" size="1.27" layer="95"/>
-<pinref part="JP1" gate="A" pin="4"/>
 </segment>
 <segment>
 <wire x1="170.18" y1="83.82" x2="170.18" y2="76.2" width="0.1524" layer="91"/>
 <label x="170.18" y="83.82" size="1.778" layer="95"/>
-<pinref part="JP2" gate="A" pin="4"/>
+<pinref part="JP1" gate="A" pin="4"/>
 </segment>
 </net>
@@
 <wire x1="104.14" y1="91.44" x2="111.76" y2="91.44" width="0.1524" layer="91"/>
 <label x="101.6" y="91.44" size="1.27" layer="95"/>
-<pinref part="JP1" gate="A" pin="5"/>
+<pinref part="JP3" gate="G$1" pin="1"/>
 </segment>
 <segment>
@@
 <net name="PGD" class="0">
 <segment>
-<wire x1="104.14" y1="99.06" x2="111.76" y2="99.06" width="0.1524" layer="91"/>
-<label x="101.6" y="99.06" size="1.27" layer="95"/>
-<pinref part="JP1" gate="A" pin="2"/>
-</segment>
-<segment>
 <pinref part="IC2" gate="G$1" pin="RA0/D+"/>
 <wire x1="162.56" y1="73.66" x2="106.68" y2="73.66" width="0.1524" layer="91"/>
 <label x="119.38" y="73.66" size="1.778" layer="95"/>
 <wire x1="162.56" y1="73.66" x2="162.56" y2="83.82" width="0.1524" layer="91"/>
-<pinref part="JP2" gate="A" pin="2"/>
 <wire x1="162.56" y1="83.82" x2="167.64" y2="83.82" width="0.1524" layer="91"/>
 <wire x1="167.64" y1="83.82" x2="167.64" y2="76.2" width="0.1524" layer="91"/>
+<pinref part="JP1" gate="A" pin="2"/>
 </segment>
 </net>
 <net name="PGC" class="0">
-<segment>
-<wire x1="104.14" y1="101.6" x2="111.76" y2="101.6" width="0.1524" layer="91"/>
-<label x="101.6" y="101.6" size="1.27" layer="95"/>
-<pinref part="JP1" gate="A" pin="1"/>
-</segment>
 <segment>
 <wire x1="162.56" y1="71.12" x2="106.68" y2="71.12" width="0.1524" layer="91"/>
@@
 <pinref part="IC2" gate="G$1" pin="RA1/D-"/>
 <wire x1="162.56" y1="71.12" x2="162.56" y2="60.96" width="0.1524" layer="91"/>
-<pinref part="JP2" gate="A" pin="1"/>
 <wire x1="162.56" y1="60.96" x2="167.64" y2="60.96" width="0.1524" layer="91"/>
 <wire x1="167.64" y1="60.96" x2="167.64" y2="68.58" width="0.1524" layer="91"/>
+<pinref part="JP1" gate="A" pin="1"/>
 </segment>
 </net>
@@
 <net name="N$3" class="0">
 <segment>
-<pinref part="JP2" gate="A" pin="6"/>
+<pinref part="JP1" gate="A" pin="6"/>
 <wire x1="172.72" y1="76.2" x2="172.72" y2="81.28" width="0.1524" layer="91"/>
-<wire x1="172.72" y1="81.28" x2="177.8" y2="81.28" width="0.1524" layer="91"/>
-<wire x1="177.8" y1="81.28" x2="177.8" y2="63.5" width="0.1524" layer="91"/>
-<wire x1="177.8" y1="63.5" x2="172.72" y2="63.5" width="0.1524" layer="91"/>
-<pinref part="JP2" gate="A" pin="5"/>
-<wire x1="172.72" y1="63.5" x2="172.72" y2="68.58" width="0.1524" layer="91"/>
-</segment>
-</net>
+<pinref part="JP1" gate="A" pin="8"/>
+<wire x1="172.72" y1="81.28" x2="175.26" y2="81.28" width="0.1524" layer="91"/>
+<wire x1="175.26" y1="81.28" x2="175.26" y2="76.2" width="0.1524" layer="91"/>
+</segment>
+</net>
+<net name="N$5" class="0">
+<segment>
+<pinref part="JP1" gate="A" pin="5"/>
+<wire x1="172.72" y1="68.58" x2="172.72" y2="63.5" width="0.1524" layer="91"/>
+<pinref part="JP1" gate="A" pin="7"/>
+<wire x1="172.72" y1="63.5" x2="175.26" y2="63.5" width="0.1524" layer="91"/>
+<wire x1="175.26" y1="63.5" x2="175.26" y2="68.58" width="0.1524" layer="91"/>
+</segment>
+</net>

Commit message: Añado splitter
Parts:
- removed C4: 22p, SparkFun:CAP0805
- removed JP3: (no value), pinhead:PINHD-1X1
- removed R11, R3, R5, R6, R7, R9: 100R, SparkFun:RESISTOR0805-RES
- removed R13, R15, R16: 220R, SparkFun:RESISTOR0805-RES
- removed X1: 53047-06, con-molex:53047-06
- added C1: 4.7u, rcl:C-EUC0805
- added JTAG: (no value), pinhead:PINHD-1X6
- added KEYB: (no value), pinhead:PINHD-1X3
- added PWUSB: MICROUSB, zxuno_rev_mcleod:MICROUSB
- added R1: 10K, rcl:R-EU_R0805
- added R2: 100R, rcl:R-EU_R0805
- C2: value 4.7u -> 22p; device SparkFun:CAP0805 -> rcl:C-EUC0805
- C3: device SparkFun:CAP0805 -> rcl:C-EUC0805
- C5: device rcl:C-USC0603K -> rcl:C-USC0805
- JP1: device pinhead:PINHD-2X4 -> pinhead:PINHD-1X5
Connections:
- removed net N$13: IC2.RC7/AN9, R5.2
- removed net N$16: IC2.RB6, R11.1
- removed net N$2: IC2.RC1/AN5, R7.2
- removed net N$3: JP1.6, JP1.8
- removed net N$5: JP1.5, JP1.7
- removed net N$6: IC2.RC0/AN4, R6.1
- removed net N$8: IC2.RC4/P1B, R3.2
- new net 3.3V: C1.1, IC2.VDD, JP1.2, JTAG.1, R1.1
- new net CLKPS2: KEYB.1
- new net DATAPS2: KEYB.2
- net GND: now also C1.2, C2.1, JTAG.2, PWUSB.GND; no longer C2.2, C4.1, R13.2, R15.2, R16.2, X1-2.S
- net N$1: now also C3.2; no longer C4.2
- net N$4: now also C2.2; no longer C3.2
- net N$7: now also R2.1; no longer R9.2
- net PGC: now also JP1.5, PWUSB.D-; no longer JP1.1
- net PGD: now also JP1.4, PWUSB.D+; no longer JP1.2
- net TCK: now also IC2.RB6, IC2.RC0/AN4, JTAG.3; no longer R11.2, R16.1, R6.2, X1-6.S
- net TDI: now also IC2.RC4/P1B, IC2.RC7/AN9, JTAG.5; no longer R13.1, R3.1, R5.1, X1-3.S
- net TDO: now also JTAG.4, R2.2; no longer R9.1, X1-4.S
- net TMS: now also IC2.RC1/AN5, JTAG.6; no longer R15.1, R7.1, X1-5.S
- net VCC: now also KEYB.3, PWUSB.VCC; no longer C2.1, IC2.VDD, JP1.4
- net VPP: now also JP1.1, R1.2; no longer JP3.1
Other:
- moved on the sheet: C2, C3, C5
