File: hardware/max128.brd (EAGLE design)
At the start: 99.6 x 73.7 mm, 11 parts, among them IC1 REG1117, IC2 EPM7128-P100, U2 AY-3-8910, X1 SCART-F

Commit message: Añado cambios
Parts:
- removed C1, C2: (no value), rcl:C0805
- removed IC1: REG1117, burr-brown:SOT223
- added B2: (no value), rectifier:1KAB
- added C7, C8: 22pF, rcl:C0805K
- added J1: (no value), dp_devices:DC_BARREL_JACK_PTH_2MM_2
- added R56: 2K, rcl:R0805
- added R65: 1M, rcl:R0805
- added U$3: DC-DC-STEP-DOWN-LM2596, diy-modules:DC-DC-STEP-DOWN-LM2596
- added U1: SN74LVC2G04DBV, 74LV:SOT23-6
- added Y1: 14.000M, crystal:HC49/S
- moved U2 15.8 mm to (88.7, 20.5)
- moved U$2 13.2 mm to (66.9, 29.3), turned to 90 degrees
- moved X1 1.70 mm to (43.7, 69.0)
Connections:
- removed net +3V3: C2.1, IC1.2
- new net 14MHZ: U1.6
- new net N$1: B2.AC1, J1.P1
- new net N$2: B2.AC2, J1.P2, J1.P3
- new net N$24: C7.1, R65.2, U1.3, Y1.2
- new net N$27: R56.1, R65.1, U1.1, U1.4
- new net N$3: B2.+, U$3.IN+
- new net N$4: B2.-, U$3.IN-
- new net N$61: C8.1, R56.2, Y1.1
- net +5V: no longer C1.1, IC1.3
- net GND: now also C7.2, C8.2, U$3.OUT-, U1.2; no longer C1.2, C2.2, IC1.1
- net VCC: now also U$3.OUT+, U1.5
Routing:
- net N$1: track 0.00 -> 18.9 mm
- net N$2: track 0.00 -> 11.6 mm
