File: hardware/addons_zxuno/wifi.brd (EAGLE design)
At the start: 31.6 x 28.3 mm, 6 parts

Commit message: Actualizo addon wifi
Parts:
- removed JP1: (no value), jumper:JP1
- added IC3: DS2431, 1wire:TO92-
- added R1: 10K, rcl:R0805
- moved MDL1 6.35 mm to (13.8, 1.98)
- moved R37 1.75 mm to (2.70, 17.1)
Connections:
- removed net VIN: JP1.2, MDL1.17, MDL1.18, MDL1.3, MDL1.8
- new net N$6: IC3.2, J11.2
- net 3.3V: now also MDL1.17, MDL1.18, MDL1.3, MDL1.8, R1.2; no longer JP1.1
- net GND: now also IC3.1
- net N$5: now also R1.1; no longer J11.8
Routing:
- net 3.3V: track 20.3 -> 66.5 mm
- net VIN: track 39.2 -> 0.00 mm
- net GND: track 39.5 -> 67.8 mm
- net N$6: track 0.00 -> 20.7 mm
- net N$2: track 30.8 -> 24.1 mm
- net N$1: track 10.8 -> 16.5 mm
- net N$5: track 35.5 -> 36.6 mm, vias 0 -> 2
- net N$3: track 7.16 -> 8.17 mm
- net N$4: track 7.38 -> 7.91 mm
