File: hardware/addons_zxuno/wifi.sch (EAGLE design)
At the start: 6 parts

Commit message: Actualizo addon wifi
Parts:
- removed JP1: (no value), jumper:JP1E
- added IC3: DS2431, 1wire:DS2431
- added R1: 10K, rcl:R-US_R0805
Connections:
- removed net VIN: JP1.2, MDL1.CH_PD, MDL1.GPIO0, MDL1.GPIO2, MDL1.VCC
- new net N$6: IC3_1W.1W, J11.2
- net 3.3V: now also MDL1.CH_PD, MDL1.GPIO0, MDL1.GPIO2, MDL1.VCC, R1.2; no longer JP1.1
- net N$5: now also R1.1; no longer J11.8
Changed lines of the file:
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@@
 <?xml version="1.0" encoding="utf-8"?>
 <!DOCTYPE eagle SYSTEM "eagle.dtd">
-<eagle version="7.3.0">
+<eagle version="9.0.0">
 <drawing>
 <settings>
 <setting alwaysvectorfont="no"/>
+<setting keepoldvectorfont="yes"/>
 <setting verticaltext="up"/>
 </settings>
@@
 <layer number="56" name="wert" color="7" fill="1" visible="no" active="no"/>
 <layer number="57" name="tCAD" color="7" fill="1" visible="no" active="no"/>
+<layer number="88" name="SimResults" color="9" fill="1" visible="yes" active="yes"/>
+<layer number="89" name="SimProbes" color="9" fill="1" visible="yes" active="yes"/>
 <layer number="90" name="Modules" color="7" fill="1" visible="no" active="yes"/>
 <layer number="91" name="Nets" color="2" fill="1" visible="yes" active="yes"/>
@@
 <part name="R37" library="rcl" deviceset="R-US_" device="R0805" value="10K"/>
 <part name="GND4" library="supply1" deviceset="GND" device=""/>
-<part name="JP1" library="jumper" deviceset="JP1E" device=""/>
+<part name="R1" library="rcl" deviceset="R-US_" device="R0805" value="10K"/>
+<part name="IC3" library="1wire" deviceset="DS2431" device="" value="DS2431"/>
 </parts>
 <sheets>
@@
 </instance>
 <instance part="GND4" gate="1" x="99.06" y="38.1"/>
-<instance part="JP1" gate="A" x="43.18" y="104.14" rot="R270"/>
+<instance part="R1" gate="G$1" x="45.72" y="68.58" smashed="yes" rot="R90">
+<attribute name="NAME" x="49.3014" y="69.85" size="1.778" layer="95" rot="R90"/>
+<attribute name="VALUE" x="49.022" y="64.77" size="1.778" layer="96" rot="R90"/>
+</instance>
+<instance part="IC3" gate="G$1" x="-12.7" y="101.6" smashed="yes">
+<attribute name="NAME" x="-6.985" y="102.235" size="1.778" layer="95"/>
+<attribute name="VALUE" x="-6.985" y="99.695" size="1.778" layer="96"/>
+</instance>
+<instance part="IC3" gate="_1W" x="7.62" y="101.6" smashed="yes" rot="R180">
+<attribute name="NAME" x="16.51" y="99.695" size="1.778" layer="95" font="vector" rot="R180"/>
+</instance>
 </instances>
 <busses>
@@
 <segment>
 <pinref part="J11" gate="G$1" pin="1"/>
-<wire x1="68.58" y1="116.84" x2="40.64" y2="116.84" width="0.1524" layer="91"/>
+<wire x1="68.58" y1="116.84" x2="45.72" y2="116.84" width="0.1524" layer="91"/>
 <label x="58.42" y="116.84" size="1.778" layer="95"/>
-<pinref part="JP1" gate="A" pin="1"/>
-<wire x1="40.64" y1="116.84" x2="40.64" y2="104.14" width="0.1524" layer="91"/>
-</segment>
-</net>
-<net name="N$1" class="0">
-<segment>
-<pinref part="MDL1" gate="G$1" pin="GPIO15"/>
-<pinref part="R37" gate="G$1" pin="1"/>
-<wire x1="78.74" y1="48.26" x2="83.82" y2="48.26" width="0.1524" layer="91"/>
-</segment>
-</net>
-<net name="VIN" class="0">
-<segment>
 <pinref part="MDL1" gate="G$1" pin="VCC"/>
+<wire x1="45.72" y1="116.84" x2="40.64" y2="116.84" width="0.1524" layer="91"/>
 <wire x1="40.64" y1="45.72" x2="45.72" y2="45.72" width="0.1524" layer="91"/>
 <pinref part="MDL1" gate="G$1" pin="GPIO0"/>
@@
 <junction x="81.28" y="53.34"/>
 <junction x="81.28" y="50.8"/>
-<pinref part="JP1" gate="A" pin="2"/>
-<wire x1="40.64" y1="101.6" x2="40.64" y2="58.42" width="0.1524" layer="91"/>
+<wire x1="40.64" y1="116.84" x2="40.64" y2="58.42" width="0.1524" layer="91"/>
 <pinref part="MDL1" gate="G$1" pin="CH_PD"/>
 <wire x1="40.64" y1="58.42" x2="40.64" y2="45.72" width="0.1524" layer="91"/>
 <wire x1="45.72" y1="58.42" x2="40.64" y2="58.42" width="0.1524" layer="91"/>
 <junction x="40.64" y="58.42"/>
+<pinref part="R1" gate="G$1" pin="2"/>
+<wire x1="45.72" y1="73.66" x2="45.72" y2="116.84" width="0.1524" layer="91"/>
+<junction x="45.72" y="116.84"/>
+</segment>
+</net>
+<net name="N$1" class="0">
+<segment>
+<pinref part="MDL1" gate="G$1" pin="GPIO15"/>
+<pinref part="R37" gate="G$1" pin="1"/>
+<wire x1="78.74" y1="48.26" x2="83.82" y2="48.26" width="0.1524" layer="91"/>
 </segment>
 </net>
@@
 <net name="N$5" class="0">
 <segment>
-<pinref part="J11" gate="G$1" pin="8"/>
 <pinref part="MDL1" gate="G$1" pin="REST"/>
-<wire x1="68.58" y1="99.06" x2="45.72" y2="99.06" width="0.1524" layer="91"/>
-<wire x1="45.72" y1="99.06" x2="45.72" y2="63.5" width="0.1524" layer="91"/>
-</segment>
-</net>
+<pinref part="R1" gate="G$1" pin="1"/>
+</segment>
+</net>
+<net name="N$6" class="0">
+<segment>
+<pinref part="J11" gate="G$1" pin="2"/>
+<pinref part="IC3" gate="_1W" pin="1W"/>
+<wire x1="68.58" y1="114.3" x2="12.7" y2="114.3" width="0.1524" layer="91"/>
+<wire x1="12.7" y1="114.3" x2="12.7" y2="101.6" width="0.1524" layer="91"/>
+</segment>
+</net>
